File: FootVibrator.brd (EAGLE design)
At the start: 30 x 44.2 mm, 43 parts, among them Q2 S9013, SW1 B3U-1000P-2P-SMD, SW2 B3U-1000P-2P-SMD, U2 ADXL345BCCZ-RL, Y1 3.2768KHZ

Commit message: update
Parts:
- removed U$10: SM06B-SRSS-TB, SH:SM06B-SRSS-TB
- removed U$11, U$12: 05FH-SM1-TB, FH:05FH-SM1-TB
- removed U$2: STM32L051K8, micro-stm:LQFP32
- removed U$3, U$4: SM04B-NSHSS-TB, NSH:SM04B-NSHSS-TB
- removed U$7, U$8: SM02B-NSHSS-TB, NSH:SM02B-NSHSS-TB
- added J1, J2: SM04B-NSHSS-TB, FootVibrator:SM04B-NSHSS-TB
- added J3: SM06B-SRSS-TB, FootVibrator:SM06B-SRSS-TB
- added J4, J5: 5051100592, FootVibrator:5051100592
- added J6, J7: SM02B-NSHSS-TB, FootVibrator:SM02B-NSHSS-TB
- added U3: STM32L051K8, FootVibrator:LQFP32
- C1, C10, C15, C16, C17, C2, C6, C8, C9: device OPL_Capacitor:C0603 -> FootVibrator:C0603
- D2, D3, D4, D5, D6: device OPL_Optoelectronics:LED-0805 -> FootVibrator:LED-0805
- D7: device OPL_Discrete_Semiconductor:DO-214AC -> FootVibrator:DO-214AC
- Q2: device OPL_Discrete_Semiconductor:SOT-23 -> FootVibrator:SOT-23
- R1, R10, R13, R14, R2, R3, R4, R5, R6, R7, R8, R9: device OPL_Resistor:R0603 -> FootVibrator:R0603
- REG1: device regulator:NJM2884-SOT-89-5 -> FootVibrator:NJM2884-SOT-89-5
- SW1, SW2: device OPL_Switch:SW2-2.6-3.0X2.5X1.2+0.4MM -> FootVibrator:SW2-2.6-3.0X2.5X1.2+0.4MM
- U2: device OPL_Sensor-Transducer:LGA14-0.8-5.0X3.0MM -> FootVibrator:LGA14-0.8-5.0X3.0MM
- U4: value NJM2716 -> TSV911AILT
- Y1: device OPL_Crystal Oscillator:X2-SMD-L2.0X1.2X0.55MM -> FootVibrator:X2-SMD-L2.0X1.2X0.55MM
- renumbered U$1 to U1, U$5 to U4
Connections:
- net +3V3: now also J3.5, J4.2, J5.4, J6.P$1, J7.P$2, U3.1, U3.17, U3.5; no longer U$10.5, U$11.4, U$12.2, U$2.1, U$2.17, U$2.5, U$7.P$2, U$8.P$1
- net +5V: now also J1.P$2, J2.P$3; no longer U$3.P$3, U$4.P$2
- net GND: now also J1.P$1, J2.P$4, J3.1, J3.4, J4.1, J4.5, J5.1, J5.5, U3.16, U3.32; no longer U$10.1, U$10.4, U$11.1, U$11.5, U$12.1, U$12.5, U$2.16, U$2.32, U$3.P$4, U$4.P$1
- net I2C1_SCL: now also J4.4, J5.2, U3.29; no longer U$11.2, U$12.4, U$2.29
- net I2C1_SDA: now also J4.3, J5.3, U3.30; no longer U$11.3, U$12.3, U$2.30
- net N$1: now also U3.31; no longer U$2.31
- net N$11: now also U3.4; no longer U$2.4
- net OCC_IN: now also U3.2; no longer U$2.2
- net OCC_OUT: now also U3.3; no longer U$2.3
- net PWM_OUT: now also U3.7; no longer U$2.7
- net RAW_FSR: now also J7.P$1; no longer U$7.P$1
- net RAW_MOTOR: now also J6.P$2; no longer U$8.P$2
- net SIGNAL_FSR: now also U3.6; no longer U$2.6
- net SPI1_CS: now also U3.14; no longer U$2.14
- net SPI1_MISO: now also U3.12; no longer U$2.12
- net SPI1_MOSI: now also U3.13; no longer U$2.13
- net SPI1_SCK: now also U3.11; no longer U$2.11
- net SYS_SWCLK: now also J3.2, U3.24; no longer U$10.2, U$2.24
- net SYS_SWDIO: now also J3.3, U3.23; no longer U$10.3, U$2.23
- net USART1_RX: now also J2.P$1, U3.20; no longer U$2.20, U$3.P$1
- net USART1_TX: now also J2.P$2, U3.19; no longer U$2.19, U$3.P$2
- net USART2_RX: now also J1.P$3, U3.9; no longer U$2.9, U$4.P$3
- net USART2_TX: now also J1.P$4, U3.8; no longer U$2.8, U$4.P$4
Other:
- board text added: "JSK Vibrator v1"
