File: FootVibrator.sch (EAGLE design)
At the start: 49 parts, among them Q1 MMBT3904, Q2 FA-128, U1 LSM9DS1

Commit message: SeeedOPLを使用するように変更
Parts:
- removed C5: 0.1 uF, rcl:C-EUC0402
- removed C7: 100 nF, rcl:C-EUC0402
- removed D1: ES1D, ES1D:ES1D
- removed LED1: GREEN, led:LEDCHIP-LED0603
- removed LED2, LED4: RED, led:LEDCHIP-LED0603
- removed LED3, LED5: YELLOW, led:LEDCHIP-LED0603
- removed Q1: MMBT3904, MMBT3904:MMBT3904
- removed R11, R12: 1k, rcl:R-EU_R0402
- removed U$6: SM04B-NSHSS-TB, NSH:SM04B-NSHSS-TB
- removed U$9: NJM2716, MyLibrary:NJM2716
- added C16, C17: 12pf, OPL_Capacitor:CERAMIC-12PF-50V-5%-NPO(0603)
- added D2: GREEN-0603, OPL_Optoelectronics:SMD-LED-CLEAR-GREEN(0603)
- added D3, D5: YELLOW-0805, OPL_Optoelectronics:SMD-LED-CLEAR-YELLOW(0805)
- added D4, D6: RED-0805, OPL_Optoelectronics:SMD-LED-CLEAR-RED(0805)
- added D7: 1N4007, OPL_Discrete_Semiconductor:DIODE-GEN-PURPOSE-1KV-1A(DO-214AC)
- added R13: 10K, OPL_Resistor:SMD-RES-10K-1%-1/10W(0603)
- added R14: 1K 1/10W, OPL_Resistor:SMD-RES-1K-5%-1/10W(0603)
- added SW1, SW2: B3U-1000P-2P-SMD, OPL_Switch:SMD-BUTTON(2P-3.0X2.5X1.2+0.4MM)-B3U-1000P-2P-SMD
- added Y1: 3.2768KHZ, OPL_Crystal Oscillator:SMD-CRYSTAL-32.768KHZ-12.5PF-20PPM-90K(2P-L2.0X1.2MM)
- C1, C12, C14, C9: value 100 nF -> 100nf; device rcl:C-EUC0402 -> OPL_Capacitor:CERAMIC-100NF-50V-10%-X7R(0603)
- C10: value 100 nF -> 100pf; device rcl:C-EUC0402 -> OPL_Capacitor:CERAMIC-100PF-50V-5%-NPO(0603)
- C11: value 10 uF -> 10UF 6.3V; device rcl:C-EUC0402 -> OPL_Capacitor:CERAMIC-10UF-6.3V-20%-X5R(0603)
- C13: value 10 nF (16V) -> 10nf; device rcl:C-EUC0402 -> OPL_Capacitor:CERAMIC-10NF-50V-10%-X7R(0603)
- C15: value 0.1 uF -> 100nf; device rcl:C-EUC0402 -> OPL_Capacitor:CERAMIC-100NF-50V-10%-X7R(0603)
- C2: value 4.7 uF -> 4.7uf; device rcl:C-EUC0402 -> OPL_Capacitor:CERAMIC-4.7UF-10V-10%-X5R(0603)
- C3: value 12 pF -> 100nf; device rcl:C-EUC0402 -> OPL_Capacitor:CERAMIC-100NF-50V-10%-X7R(0603)
- C4: value 12 pF -> 1uf; device rcl:C-EUC0402 -> OPL_Capacitor:CERAMIC-1UF-25V-10%-X7R(0603)
- C6: value 1 uF -> 100nf; device rcl:C-EUC0402 -> OPL_Capacitor:CERAMIC-100NF-50V-10%-X7R(0603)
- C8: value 1 uF -> 1uf; device rcl:C-EUC0402 -> OPL_Capacitor:CERAMIC-1UF-25V-10%-X7R(0603)
- Q2: value FA-128 -> S9013; device crystal:FA-128 -> OPL_Discrete_Semiconductor:SMD-TRANSISTORS-NPN-25V-500MA-S9013(SOT-23)
- R1, R3, R4: value 1.5k -> 1.5K 1/10W; device rcl:R-EU_R0402 -> OPL_Resistor:SMD-RES-1.5K-5%-1/10W(0603)
- R10, R7, R8, R9: value 1k -> 1K 1/10W; device rcl:R-EU_R0402 -> OPL_Resistor:SMD-RES-1K-5%-1/10W(0603)
- R2: value 100k -> 1K 1/10W; device rcl:R-EU_R0402 -> OPL_Resistor:SMD-RES-1K-5%-1/10W(0603)
- R5: value 10k -> 100K 1/10W; device rcl:R-EU_R0402 -> OPL_Resistor:SMD-RES-100K-5%-1/10W(0603)
- R6: value 10k -> 10K; device rcl:R-EU_R0402 -> OPL_Resistor:SMD-RES-10K-1%-1/10W(0603)
- U$4: value SKRPACE010 -> SM04B-NSHSS-TB; device MyLibrary:SKRPACE010 -> NSH:SM04B-NSHSS-TB
- U$5: value SKRPACE010 -> NJM2716; device MyLibrary:SKRPACE010 -> FootVibrator:NJM2716
Connections:
- removed net N$10: LED5.A, R12.1
- removed net N$9: LED4.A, R11.1
- removed net NRST: C5.1, U$2.NRST, U$5.B
- new net N$11: C6.2, SW1.2, U$2.NRST
- new net N$12: D4.+, R14.1
- net +3V3: now also C3.2, C4.2, D7.-, R14.2, R2.2, R5.1, U$5.V+; no longer C6.1, C7.1, D1.C, R11.2, R12.2, R2.1, U$9.V+
- net +5V: now also U$4.2; no longer U$6.2
- net GND: now also C16.1, C17.1, C3.1, C4.1, C6.1, D2.-, Q2.E, R13.1, SW1.1, U$4.1, U$5.GND; no longer C3.2, C4.2, C5.2, C6.2, C7.2, LED1.C, Q1.E, Q2.2, Q2.4, R5.1, U$5.A, U$6.1, U$9.GND
- net N$1: now also R5.2, SW2.2; no longer R2.2, U$4.B
- net N$2: now also D3.+, R2.1; no longer R5.2, U$4.A
- net N$3: now also D2.+; no longer LED1.A
- net N$6: now also Q2.B; no longer Q1.B
- net N$7: now also D5.+; no longer LED2.A
- net N$8: now also D6.+; no longer LED3.A
- net OCC_IN: now also C16.2, Y1.1; no longer C3.1, Q2.1
- net OCC_OUT: now also C17.2, Y1.2; no longer C4.1, Q2.3
- net RAW_FSR: now also U$5.+; no longer U$9.+
- net RAW_MOTOR: now also D7.+, Q2.C; no longer D1.A, Q1.C
- net SIGNAL_FSR: now also U$5.-, U$5.OUT; no longer U$9.-, U$9.OUT
- net USART1_RX: now also D6.-; no longer LED4.C
- net USART1_TX: now also D5.-; no longer LED5.C
- net USART2_RX: now also D4.-, U$4.3; no longer LED2.C, U$6.3
- net USART2_TX: now also D3.-, U$4.4; no longer LED3.C, U$6.4
Other:
- moved on the sheet: R10, R2, R5, R8, R9, U$3

Commit message: コンデンサの数を減らした
Parts:
- removed C11: 10UF 6.3V, OPL_Capacitor:CERAMIC-10UF-6.3V-20%-X5R(0603)
- removed C2: 4.7uf, OPL_Capacitor:CERAMIC-4.7UF-10V-10%-X5R(0603)
- removed C3: 100nf, OPL_Capacitor:CERAMIC-100NF-50V-10%-X7R(0603)
- removed C4: 1uf, OPL_Capacitor:CERAMIC-1UF-25V-10%-X7R(0603)
Connections:
- net +3V3: no longer C11.1, C2.1, C3.2, C4.2
- net GND: no longer C11.2, C2.2, C3.1, C4.1
Other:
- moved on the sheet: C10

Commit message: アートワーク引き直した
Parts:
- removed C12, C14: 100nf, OPL_Capacitor:CERAMIC-100NF-50V-10%-X7R(0603)
- removed C13: 10nf, OPL_Capacitor:CERAMIC-10NF-50V-10%-X7R(0603)
- removed U1: LSM9DS1, LSM9DS1:LSM9DS1
- added C2: 100nf, OPL_Capacitor:CERAMIC-100NF-50V-10%-X7R(0603)
- added U2: ADXL345BCCZ-RL, OPL_Sensor-Transducer:MOTION/POSITION-ADXL345BCCZ-RL(14P-5.0X3.0MM)
- D2: value GREEN-0603 -> GREEN-0805; device OPL_Optoelectronics:SMD-LED-CLEAR-GREEN(0603) -> OPL_Optoelectronics:SMD-LED-CLEAR-GREEN(0805)
- U$1: device MyLibrary:VL53L0X -> FootVibrator:VL53L0X
- U$2: value STM32L071K8 -> STM32L051K8; device micro-stm:STM32L071K8 -> micro-stm:STM32L051K8
Connections:
- removed net N$4: C13.1, U1.CAP
- removed net N$5: C14.1, U1.C1
- removed net SPI1_CS_AG: U$2.PB0, U1.CS_A/G
- removed net SPI1_CS_M: U$2.PB1, U1.CS_M
- new net N$3: R13.2, SW2.1
- new net SPI1_CS: U$2.PB0, U2.!CS
- net +3V3: now also C2.1, U2.VDDI/O, U2.VS; no longer C12.1, U$2.VDDIO, U1.VDD, U1.VDDIO
- net GND: now also C2.2, U2.GND@1, U2.GND@2, U2.GND@3; no longer C12.2, C13.2, C14.2, U$2.VSSA, U1.GND, U1.RES
- net SPI1_MISO: now also U2.SDO/ALTADDRESS; no longer U1.SDO_A/G, U1.SDO_M
- net SPI1_MOSI: now also U2.SDA/SDI/SDIO; no longer U1.SDA/SDI/SDO
- net SPI1_SCK: now also U2.SCL/SCLK; no longer U1.SCL/SPC

Commit message: update
Parts:
- removed U$10: SM06B-SRSS-TB, SH:SM06B-SRSS-TB
- removed U$11, U$12: 05FH-SM1-TB, FH:05FH-SM1-TB
- removed U$2: STM32L051K8, micro-stm:STM32L051K8
- removed U$3, U$4: SM04B-NSHSS-TB, NSH:SM04B-NSHSS-TB
- removed U$5: NJM2716, FootVibrator:NJM2716
- removed U$7, U$8: SM02B-NSHSS-TB, NSH:SM02B-NSHSS-TB
- added J1, J2: SM04B-NSHSS-TB, FootVibrator:SM04B-NSHSS-TB
- added J3: SM06B-SRSS-TB, FootVibrator:SM06B-SRSS-TB
- added J4, J5: 5051100592, FootVibrator:5051100592
- added J6, J7: SM02B-NSHSS-TB, FootVibrator:SM02B-NSHSS-TB
- added U3: STM32L051K8, FootVibrator:STM32L051K8
- added U4: TSV911AILT, FootVibrator:TSV911AILT
- C1, C15, C2, C6, C9: device OPL_Capacitor:CERAMIC-100NF-50V-10%-X7R(0603) -> FootVibrator:CERAMIC-100NF-50V-10%-X7R(0603)
- C10: device OPL_Capacitor:CERAMIC-100PF-50V-5%-NPO(0603) -> FootVibrator:CERAMIC-100PF-50V-5%-NPO(0603)
- C16, C17: device OPL_Capacitor:CERAMIC-12PF-50V-5%-NPO(0603) -> FootVibrator:CERAMIC-12PF-50V-5%-NPO(0603)
- C8: device OPL_Capacitor:CERAMIC-1UF-25V-10%-X7R(0603) -> FootVibrator:CERAMIC-1UF-25V-10%-X7R(0603)
- D2: device OPL_Optoelectronics:SMD-LED-CLEAR-GREEN(0805) -> FootVibrator:SMD-LED-CLEAR-GREEN(0805)
- D3, D5: device OPL_Optoelectronics:SMD-LED-CLEAR-YELLOW(0805) -> FootVibrator:SMD-LED-CLEAR-YELLOW(0805)
- D4, D6: device OPL_Optoelectronics:SMD-LED-CLEAR-RED(0805) -> FootVibrator:SMD-LED-CLEAR-RED(0805)
- D7: device OPL_Discrete_Semiconductor:DIODE-GEN-PURPOSE-1KV-1A(DO-214AC) -> FootVibrator:DIODE-GEN-PURPOSE-1KV-1A(DO-214AC)
- Q2: device OPL_Discrete_Semiconductor:SMD-TRANSISTORS-NPN-25V-500MA-S9013(SOT-23) -> FootVibrator:SMD-TRANSISTORS-NPN-25V-500MA-S9013(SOT-23)
- R1, R3, R4: device OPL_Resistor:SMD-RES-1.5K-5%-1/10W(0603) -> FootVibrator:SMD-RES-1.5K-5%-1/10W(0603)
- R10, R14, R2, R7, R8, R9: device OPL_Resistor:SMD-RES-1K-5%-1/10W(0603) -> FootVibrator:SMD-RES-1K-5%-1/10W(0603)
- R13, R6: device OPL_Resistor:SMD-RES-10K-1%-1/10W(0603) -> FootVibrator:SMD-RES-10K-1%-1/10W(0603)
- R5: device OPL_Resistor:SMD-RES-100K-5%-1/10W(0603) -> FootVibrator:SMD-RES-100K-5%-1/10W(0603)
- REG1: device regulator:NJM2884 -> FootVibrator:NJM2884
- SW1, SW2: device OPL_Switch:SMD-BUTTON(2P-3.0X2.5X1.2+0.4MM)-B3U-1000P-2P-SMD -> FootVibrator:SMD-BUTTON(2P-3.0X2.5X1.2+0.4MM)-B3U-1000P-2P-SMD
- U2: device OPL_Sensor-Transducer:MOTION/POSITION-ADXL345BCCZ-RL(14P-5.0X3.0MM) -> FootVibrator:MOTION/POSITION-ADXL345BCCZ-RL(14P-5.0X3.0MM)
- Y1: device OPL_Crystal Oscillator:SMD-CRYSTAL-32.768KHZ-12.5PF-20PPM-90K(2P-L2.0X1.2MM) -> FootVibrator:SMD-CRYSTAL-32.768KHZ-12.5PF-20PPM-90K(2P-L2.0X1.2MM)
- renumbered U$1 to U1
Connections:
- net +3V3: now also J3.5, J4.2, J5.4, J6.1, J7.2, U3.VDD, U3.VDDA, U4.V+; no longer U$10.5, U$11.4, U$12.2, U$2.VDD, U$2.VDDA, U$5.V+, U$7.2, U$8.1
- net +5V: now also J1.2, J2.3; no longer U$3.3, U$4.2
- net GND: now also J1.1, J2.4, J3.1, J3.4, J4.1, J4.5, J5.1, J5.5, U3.VSS, U4.GND; no longer U$10.1, U$10.4, U$11.1, U$11.5, U$12.1, U$12.5, U$2.VSS, U$3.4, U$4.1, U$5.GND
- net I2C1_SCL: now also J4.4, J5.2, U3.PB6; no longer U$11.2, U$12.4, U$2.PB6
- net I2C1_SDA: now also J4.3, J5.3, U3.PB7; no longer U$11.3, U$12.3, U$2.PB7
- net N$1: now also U3.BOOT0; no longer U$2.BOOT0
- net N$11: now also U3.NRST; no longer U$2.NRST
- net OCC_IN: now also U3.OSC_IN; no longer U$2.OSC_IN
- net OCC_OUT: now also U3.OSC_OUT; no longer U$2.OSC_OUT
- net PWM_OUT: now also U3.PA1; no longer U$2.PA1
- net RAW_FSR: now also J7.1, U4.+; no longer U$5.+, U$7.1
- net RAW_MOTOR: now also J6.2; no longer U$8.2
- net SIGNAL_FSR: now also U3.PA0-WKUP, U4.-, U4.OUT; no longer U$2.PA0-WKUP, U$5.-, U$5.OUT
- net SPI1_CS: now also U3.PB0; no longer U$2.PB0
- net SPI1_MISO: now also U3.PA6; no longer U$2.PA6
- net SPI1_MOSI: now also U3.PA7; no longer U$2.PA7
- net SPI1_SCK: now also U3.PA5; no longer U$2.PA5
- net SYS_SWCLK: now also J3.2, U3.PA14; no longer U$10.2, U$2.PA14
- net SYS_SWDIO: now also J3.3, U3.PA13; no longer U$10.3, U$2.PA13
- net USART1_RX: now also J2.1, U3.PA10; no longer U$2.PA10, U$3.1
- net USART1_TX: now also J2.2, U3.PA9; no longer U$2.PA9, U$3.2
- net USART2_RX: now also J1.3, U3.PA3; no longer U$2.PA3, U$4.3
- net USART2_TX: now also J1.4, U3.PA2; no longer U$2.PA2, U$4.4
